File: Board/LaserBoardv1.0.sch (EAGLE design)
At the start: 62 parts, among them IC1 L293D, IC2 L293D, IC3 L293D, IC4 4050D, J2 ICSP, Q1 1A/60V/500mΩ, Q2 310mA/60V/1.6Ω, Q4 310mA/60V/1.6Ω, U1 FT231XS, U2 MIC5205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

Commit message: Board Finished
Parts:
- JP1: device jumper:JP2E -> jumper:JP4E
Connections:
- removed net SR8: U3.QH
- new net N$13: D1.A, PWR.1
- net 12V: now also JP1.1; no longer D1.A, PWR.1
- net 3.3V: now also JP1.3; no longer JP1.2
- net 5V: now also JP1.2; no longer JP1.1
- net CD: no longer JP5.8
- net DP8: no longer JP6.1, Q4.G, R12.2
- net DP9: now also JP6.1, Q4.G, R12.2
- net GND: now also JP1.4; no longer JP1.3
- net SR0: now also U3.QA
- net SR1: now also U3.QB; no longer U3.QA
- net SR2: now also U3.QC; no longer U3.QB
- net SR3: now also U3.QD; no longer U3.QC
- net SR4: now also U3.QE; no longer U3.QD
- net SR5: now also U3.QF; no longer U3.QE
- net SR6: now also U3.QG; no longer U3.QF
- net SR7: now also U3.QH; no longer U3.QG
